File: hw/pi-power-hub/pi-power-hub.kicad_sch (KiCad schematic)
At the start: 9 parts

Commit message: Updates
Parts:
- removed SW?: SW_DPST_x2, symbol Switch:SW_DPST_x2
- added C1, C2, C3, C4, C5, C6: 47nf, Capacitor_THT:C_Disc_D3.8mm_W2.6mm_P2.50mm, symbol pspice:CAP
- added J4: Conn_01x04_Male, Connector_JST:JST_PH_B4B-PH-K_1x04_P2.00mm_Vertical, symbol Connector:Conn_01x04_Male
- added J5: USB_B_Micro, Connector_USB:USB_Micro-B_Amphenol_10103594-0001LF_Horizontal, symbol Connector:USB_B_Micro
- added J8: Conn_01x02_Male, Connector_JST:JST_XH_B2B-XH-A_1x02_P2.50mm_Vertical, symbol Connector:Conn_01x02_Male
- added Q1, Q10, Q11, Q2, Q3, Q8: 2N3904, Package_TO_SOT_THT:TO-92_Inline, symbol Transistor_BJT:2N3904
- added Q12, Q13, Q4, Q5, Q6, Q9: IRFZ44NPBF, eec:Infineon_Technologies_AG-IRFZ44NPBF-0, symbol eec:IRFZ44NPBF
- added Q7: S8550, Package_TO_SOT_THT:TO-92_Inline, symbol Transistor_BJT:S8550
- added R1, R10, R12, R13, R2, R3, R7: 2k, Resistor_THT:R_Axial_DIN0207_L6.3mm_D2.5mm_P7.62mm_Horizontal, symbol Device:R
- added R11, R14, R15, R4, R5, R6: 20k, Resistor_THT:R_Axial_DIN0207_L6.3mm_D2.5mm_P7.62mm_Horizontal, symbol Device:R
- added R8: 200, Resistor_THT:R_Axial_DIN0207_L6.3mm_D2.5mm_P7.62mm_Horizontal, symbol Device:R
- added R9: 1k, Resistor_THT:R_Axial_DIN0207_L6.3mm_D2.5mm_P7.62mm_Horizontal, symbol Device:R
- added SW1, SW2, SW3, SW4, SW5, SW6: SW_Push_Dual, Button_Switch_THT:SW_PUSH_6mm_H8.5mm, symbol Switch:SW_Push
- U1: renamed from U?; footprint RPi_Pico:RPi_Pico_SMD_TH -> MCU_RaspberryPi_and_Boards:RPi_Pico_SMD_TH
- gave numbers to parts that had none: 7
Connections:
- net 5V: now reaches J3.1 (VBUS)
- net 5V: now also J1.1 (VBUS), J10.1 (VBUS), J2.1 (VBUS), J7.1 (VBUS), J9.1 (VBUS), U1.39 (VSYS), J8.1 (Pin_1), R11.1, R14.1, R15.1, R4.1, R5.1, R6.1
- net usb_dt: now reaches J3.2 (D-)
- net usb_dt: now also J1.2 (D-), J1.3 (D+), J10.2 (D-), J10.3 (D+), J2.2 (D-), J2.3 (D+), J3.3 (D+), J6.2 (D-), J6.3 (D+), J6.4 (ID), J7.2 (D-), J7.3 (D+), J9.2 (D-), J9.3 (D+), J5.2 (D-), J5.3 (D+), J5.4 (ID)
- net at J3.4 (GND): now also Q6.2 (DRAIN)
- net at J1.4 (GND): now also Q4.2 (DRAIN)
- net at J9.4 (GND): now also Q12.2 (DRAIN)
- net at J2.4 (GND): now also Q5.2 (DRAIN)
- net PORT_1_BTN: now reaches U1.10 (GPIO7)
- net PORT_1_BTN: now also SW1.2
- net PORT_2_enable: now reaches U1.11 (GPIO8)
- net PORT_2_enable: now also R12.1
- net PORT_2_BTN: now reaches U1.12 (GPIO9)
- net PORT_2_BTN: now also SW5.2
- net GND: now reaches U1.13 (GND)
- net GND: now also J6.5 (GND), U1.18 (GND), U1.23 (GND), U1.28 (GND), U1.3 (GND), U1.38 (GND), U1.8 (GND), C1.2, C2.2, C3.2, C4.2, C5.2, C6.2, J5.5 (GND), Q1.1 (E), Q10.1 (E), Q11.1 (E), Q12.3 (SOURCE), Q13.3 (SOURCE), Q2.1 (E), Q3.1 (E), Q4.3 (SOURCE), Q5.3 (SOURCE), Q6.3 (SOURCE), Q8.1 (E), Q9.3 (SOURCE), R7.1, R8.2
- net PORT_3_enable: now reaches U1.14 (GPIO10)
- net PORT_3_enable: now also R2.1
- net PORT_3_BTN: now reaches U1.15 (GPIO11)
- net PORT_3_BTN: now also SW2.2
- net at U1.19 (GPIO14): now also Q7.2 (B)
- net usb_power_in: now reaches U1.20 (GPIO15)
- net usb_power_in: now also R7.2, R9.1
- net PORT_6_BTN: now reaches U1.21 (GPIO16)
- net PORT_6_BTN: now also SW6.2
- net PORT_6_enable: now reaches U1.22 (GPIO17)
- net PORT_6_enable: now also R13.1
- net PORT_5_BTN: now reaches U1.24 (GPIO18)
- net PORT_5_BTN: now also SW4.2
- net PORT_5_enable: now reaches U1.25 (GPIO19)
- net PORT_5_enable: now also R10.1
- net PORT_4_BTN: now reaches U1.26 (GPIO20)
- net PORT_4_BTN: now also SW3.2
- net PORT_4_enable: now reaches U1.27 (GPIO21)
- net PORT_4_enable: now also R3.1
- net 3.3V: now reaches U1.36 (3V3)
- net 3.3V: now also Q7.1 (E), SW1.1, SW2.1, SW3.1, SW4.1, SW5.1, SW6.1
- net RGB_led_R: now reaches U1.4 (GPIO2)
- net RGB_led_R: now also J4.1 (Pin_1)
- net RGB_led_G: now reaches U1.5 (GPIO3)
- net RGB_led_G: now also J4.2 (Pin_2)
- net RGB_led_B: now reaches U1.6 (GPIO4)
- net RGB_led_B: now also J4.3 (Pin_3)
- net PORT_1_enable: now reaches U1.9 (GPIO6)
- net PORT_1_enable: now also R1.1
- net at J7.4 (GND): now also Q9.2 (DRAIN)
- net at J10.4 (GND): now also Q13.2 (DRAIN)
- net at J6.1 (VBUS): now also J8.2 (Pin_2)
- new net: Q2.2 (B), R2.2
- new net: Q1.2 (B), R1.2
- new net: C1.1, Q1.3 (C), Q4.1 (GATE), R4.2
- new net: Q8.2 (B), R10.2
- new net: Q11.2 (B), R13.2
- new net: C6.1, Q11.3 (C), Q13.1 (GATE), R15.2
- new net: C4.1, Q8.3 (C), Q9.1 (GATE), R11.2
- new net: C3.1, Q3.3 (C), Q6.1 (GATE), R6.2
- new net: C2.1, Q2.3 (C), Q5.1 (GATE), R5.2
- new net: C5.1, Q10.3 (C), Q12.1 (GATE), R14.2
- new net: Q10.2 (B), R12.2
- new net: Q3.2 (B), R3.2
- new net: J4.4 (Pin_4), R8.1
- new net: J5.1 (VBUS), R9.2
- new net NPN_enable: Q7.3 (C)
Other:
- note added: "PORT_1"
- note added: "PORT_2"
- note added: "PORT_3"
- note added: "PORT_4"
- note added: "PORT_5"
- note added: "PORT_6"
- note added: "USB Power in (TV detection only)"
- moved on the sheet: J1, J10, J2, J3, J6, J7, J9, U1

Commit message: Change output pins order
Connections:
- net 5V: now also J8.2 (Pin_2); no longer J8.1 (Pin_1)
- net PORT_1_BTN: now also SW2.2; no longer SW1.2
- net PORT_3_BTN: now also SW1.2; no longer SW2.2
- net 5V_Switched: now reaches J6.1 (VBUS)
- net 5V_Switched: now also J8.1 (Pin_1); no longer J8.2 (Pin_2)
Changed lines of the file:
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@@
-    (stroke (width 0) (type default) (color 0 0 0 0))
-  )
-  (wire (pts (xy 191.77 13.97) (xy 191.77 19.05))
-    (stroke (width 0) (type default) (color 0 0 0 0))
-  )
-  (wire (pts (xy 152.4 13.97) (xy 191.77 13.97))
     (stroke (width 0) (type default) (color 0 0 0 0))
   )
@@
     (stroke (width 0) (type default) (color 0 0 0 0))
   )
+  (wire (pts (xy 152.4 15.494) (xy 152.4 17.78))
+    (stroke (width 0) (type default) (color 0 0 0 0))
+  )
   (wire (pts (xy 216.916 100.33) (xy 217.805 100.33))
     (stroke (width 0) (type default) (color 0 0 0 0))
@@
   )
   (wire (pts (xy 59.69 173.482) (xy 63.5 173.482))
-    (stroke (width 0) (type default) (color 0 0 0 0))
-  )
-  (wire (pts (xy 152.4 17.78) (xy 152.4 13.97))
     (stroke (width 0) (type default) (color 0 0 0 0))
   )
@@
     )
   )
-  (global_label "PORT_1_BTN" (shape output) (at 82.042 66.294 0) (fields_autoplaced)
+  (global_label "PORT_3_BTN" (shape output) (at 82.042 66.294 0) (fields_autoplaced)
     (effects (font (size 1.27 1.27)) (justify left))
     (property "Intersheet References" "${INTERSHEET_REFS}" (id 0) (at 96.0061 66.2146 0)
@@
     )
   )
-  (global_label "PORT_3_BTN" (shape output) (at 86.106 128.016 0) (fields_autoplaced)
+  (global_label "PORT_1_BTN" (shape output) (at 86.106 128.016 0) (fields_autoplaced)
     (effects (font (size 1.27 1.27)) (justify left))
     (property "Intersheet References" "${INTERSHEET_REFS}" (id 0) (at 100.0701 127.9366 0)
@@
     )
   )
+  (global_label "5V_Switched" (shape input) (at 191.77 21.59 180) (fields_autoplaced)
+    (effects (font (size 1.27 1.27)) (justify right))
+    (property "Intersheet References" "${INTERSHEET_REFS}" (id 0) (at 177.7455 21.5106 0)
+      (effects (font (size 1.27 1.27)) (justify right) hide)
+    )
+  )
   (global_label "3.3V" (shape input) (at 257.556 121.666 180) (fields_autoplaced)
     (effects (font (size 1.27 1.27)) (justify right))
@@
     )
   )
-  (global_label "5V" (shape output) (at 191.77 21.59 180) (fields_autoplaced)
-    (effects (font (size 1.27 1.27)) (justify right))
-    (property "Intersheet References" "${INTERSHEET_REFS}" (id 0) (at 187.0588 21.5106 0)
+  (global_label "5V" (shape output) (at 191.77 19.05 180) (fields_autoplaced)
+    (effects (font (size 1.27 1.27)) (justify right))
+    (property "Intersheet References" "${INTERSHEET_REFS}" (id 0) (at 187.0588 18.9706 0)
       (effects (font (size 1.27 1.27)) (justify right) hide)
     )
@@
     )
   )
+  (global_label "5V_Switched" (shape input) (at 152.4 15.494 180) (fields_autoplaced)
+    (effects (font (size 1.27 1.27)) (justify right))
+    (property "Intersheet References" "${INTERSHEET_REFS}" (id 0) (at 138.3755 15.4146 0)
+      (effects (font (size 1.27 1.27)) (justify right) hide)
+    )
+  )
